Commit message: Adapt RVIZ and Gz windows to the new ros2srrc_hmi layout.

File: irb120cranfield_gazebo/urdf/irb120cranfield_1.urdf.xacro (robot description, xacro)
@@ -32,6 +32,4 @@
   <xacro:arg name="bringup" default="false"/>
   <xacro:property name="bringup" value="$(arg bringup)"/>
-  <xacro:arg name="hmi" default="false"/>
-  <xacro:property name="hmi" value="$(arg hmi)"/>
   <xacro:arg name="robot_ip" default="0.0.0.0"/>
   <xacro:property name="robot_ip" value="$(arg robot_ip)"/>
@@ -91,15 +89,3 @@
     <origin xyz="-0.6506 0.6489 0.8605" rpy="0.0 0.0 0.0" />
   </joint>
-  <!-- ros2srrc_HMI CAMERA -->
-  <xacro:if value="${hmi}">
-    <xacro:include filename="$(find ros2srrc_hmi)/urdf/hmicamera.urdf.xacro"/>
-    <xacro:HMI_camera
-      x="2.0"
-      y="1.25"
-      z="1.85"
-      roll="0.0"
-      pitch="0.35"
-      yaw="-2.6"
-    />
-  </xacro:if>
 </robot>

File: irb120cranfield_gazebo/urdf/irb120cranfield_2.urdf.xacro (robot description, xacro)
@@ -32,6 +32,4 @@
   <xacro:arg name="bringup" default="false"/>
   <xacro:property name="bringup" value="$(arg bringup)"/>
-  <xacro:arg name="hmi" default="false"/>
-  <xacro:property name="hmi" value="$(arg hmi)"/>
   <xacro:arg name="robot_ip" default="0.0.0.0"/>
   <xacro:property name="robot_ip" value="$(arg robot_ip)"/>
@@ -124,15 +122,3 @@
     <origin xyz="0.0 0.0 0.0" rpy="0.0 0.0 0.0" />
   </joint>
-  <!-- ros2srrc_HMI CAMERA -->
-  <xacro:if value="${hmi}">
-    <xacro:include filename="$(find ros2srrc_hmi)/urdf/hmicamera.urdf.xacro"/>
-    <xacro:HMI_camera
-      x="2.0"
-      y="1.25"
-      z="1.85"
-      roll="0.0"
-      pitch="0.35"
-      yaw="-2.6"
-    />
-  </xacro:if>
 </robot>
