Commit message: Update irb120cranfield to adapt to new changes in ros2srrc.

File: irb120cranfield/urdf/irb120cranfield_1.urdf.xacro (robot description, xacro)
@@ -29,19 +29,64 @@
 # IFRA-Cranfield (2025) ROS 2 Sim-to-Real Robot Control. ABB IRB-120 Robot. URL: https://github.com/IFRA-Cranfield/irb120_CranfieldRobotics.
 -->
-<sdf version="1.4">
-  <world name="default">
-    <!-- WORLD COMPONENTS: STANDARD -->
-    <gravity>0 0 -9.8</gravity>
-    <include>
-      <uri>model://ground_plane</uri>
-    </include>
-    <include>
-      <uri>model://sun</uri>
-    </include>
-    <scene>
-      <shadows>0</shadows>
-    </scene>
-    <!-- GAZEBO PLUGINS: -->
-    <plugin name="gazebo_link_attacher" filename="libgazebo_link_attacher.so"/>
-  </world>
-</sdf>
+<robot name="irb120" xmlns:xacro="http://ros.org/wiki/xacro">
+  <!-- PASS ARGUMENTS: -->
+  <xacro:arg name="bringup" default="false"/>
+  <xacro:property name="bringup" value="$(arg bringup)"/>
+  <xacro:arg name="robot_ip" default="0.0.0.0"/>
+  <xacro:property name="robot_ip" value="$(arg robot_ip)"/>
+  <xacro:arg name="EE" default="true"/>
+  <xacro:property name="EE" value="$(arg EE)"/>
+  <xacro:arg name="EE_name" default="none"/>
+  <xacro:property name="EE_name" value="$(arg EE_name)"/>
+  <!-- Include XACRO-MACRO file of the IRB120: -->
+  <xacro:include filename="$(find ros2srrc_robots)/irb120/urdf/irb120_macro.urdf.xacro"/>
+  <xacro:irb120
+    bringup="${bringup}"
+    robot_ip="${robot_ip}"
+    EE="${EE}"
+    EE_name="${EE_name}"
+  />
+  <!-- Load ROS 2 Gazebo Plugin -->
+  <xacro:unless value="${bringup}">
+    <gazebo>
+      <plugin filename="libgazebo_ros2_control.so" name="gazebo_ros2_control">
+        <robot_sim_type>gazebo_ros2_control/GazeboSystem</robot_sim_type>
+        <!-- IRB120 Controller -->
+        <parameters>$(find ros2srrc_robots)/irb120/config/controller.yaml</parameters>
+      </plugin>
+    </gazebo>
+  </xacro:unless>
+  <!-- World: LINK -->
+  <link name="world"/>
+  <!-- ABB IRB-120 ENCLOSURE -->
+  <link name="cell">
+    <visual>
+      <origin xyz="0.0 0.0 0.0" rpy="0 0 0" />
+      <geometry>
+        <mesh filename="file://$(find irb120cranfield)/meshes/irb120enclosure/IRB120enclosure.dae" scale="1 1 1" />
+      </geometry>
+    </visual>
+    <collision>
+      <origin xyz="0.0 0.0 0.0" rpy="0 0 0" />
+      <geometry>
+        <mesh filename="file://$(find irb120cranfield)/meshes/irb120enclosure/IRB120enclosure.dae" scale="1 1 1" />
+      </geometry>
+    </collision>
+    <inertial>
+      <mass value="1000.0"/>
+      <inertia ixx="500.0" ixy="500.0" ixz="500.0" iyy="500.0" iyz="500.0" izz="500.0" />
+    </inertial>
+  </link>
+  <!-- Robot Cell: FIXED JOINT -->
+  <joint name="world-cell-fixed" type="fixed">
+    <parent link="world"/>
+    <child link="cell"/>
+    <origin xyz="0.926 -0.124 0.0" rpy="0.0 0.0 0.0" />
+  </joint>
+  <!-- Robot+Cell JOINT -->
+  <joint name="cell-base_link-fixed" type="fixed">
+    <parent link="cell"/>
+    <child link="base_link"/>
+    <origin xyz="-0.6506 0.6489 0.8605" rpy="0.0 0.0 0.0" />
+  </joint>
+</robot>

File: irb120cranfield/urdf/irb120cranfield_2.urdf.xacro (robot description, xacro)
@@ -72,5 +72,5 @@
       <origin xyz="0.0 0.0 0.0" rpy="0 0 0" />
       <geometry>
-        <mesh filename="file://$(find irb120cranfield_gazebo)/meshes/irb120enclosure/IRB120enclosure.dae" scale="1 1 1" />
+        <mesh filename="file://$(find irb120cranfield)/meshes/irb120enclosure/IRB120enclosure.dae" scale="1 1 1" />
       </geometry>
     </visual>
@@ -78,5 +78,5 @@
       <origin xyz="0.0 0.0 0.0" rpy="0 0 0" />
       <geometry>
-        <mesh filename="file://$(find irb120cranfield_gazebo)/meshes/irb120enclosure/IRB120enclosure.dae" scale="1 1 1" />
+        <mesh filename="file://$(find irb120cranfield)/meshes/irb120enclosure/IRB120enclosure.dae" scale="1 1 1" />
       </geometry>
     </collision>
@@ -103,5 +103,5 @@
       <origin xyz="0.0 0.0 0.0" rpy="0 0 0" />
       <geometry>
-        <mesh filename="file://$(find irb120cranfield_gazebo)/meshes/irb120enclosure/ergobox.dae" scale="1 1 1" />
+        <mesh filename="file://$(find irb120cranfield)/meshes/irb120enclosure/ergobox.dae" scale="1 1 1" />
       </geometry>
     </visual>
@@ -109,5 +109,5 @@
       <origin xyz="0.0 0.0 0.0" rpy="0 0 0" />
       <geometry>
-        <mesh filename="file://$(find irb120cranfield_gazebo)/meshes/irb120enclosure/ergobox.dae" scale="1 1 1" />
+        <mesh filename="file://$(find irb120cranfield)/meshes/irb120enclosure/ergobox.dae" scale="1 1 1" />
       </geometry>
     </collision>
@@ -123,92 +123,3 @@
     <origin xyz="0.0 0.0 0.0" rpy="0.0 0.0 0.0" />
   </joint>
-  <!-- ARUCO TAG -->
-  <xacro:unless value="${bringup}">
-    <!-- ARUCO GRID -->
-    <link name="aruco_grid">
-      <visual>
-        <origin xyz="0.0 0.0 0.0" rpy="0 0 0" />
-        <geometry>
-          <mesh filename="file://$(find irb120cranfield_gazebo)/meshes/aruco/arucoGrid.dae" scale="1 1 1" />
-        </geometry>
-      </visual>
-      <collision>
-        <origin xyz="0.0 0.0 0.0" rpy="0 0 0" />
-        <geometry>
-          <mesh filename="file://$(find irb120cranfield_gazebo)/meshes/aruco/arucoGrid.dae" scale="1 1 1" />
-        </geometry>
-      </collision>
-      <inertial>
-        <mass value="10.0"/>
-        <inertia ixx="0.0002" ixy="0.0002" ixz="0.0002" iyy="0.0" iyz="0.0" izz="0.0" />
-      </inertial>
-    </link>
-    <joint name="cell-aruco_grid-fixed" type="fixed">
-      <parent link="cell"/>
-      <child link="aruco_grid"/>
-      <origin xyz="0.0 0.0 0.0" rpy="0.0 0.0 0.0" />
-    </joint>
-    <gazebo reference="cell-aruco_grid-fixed">
-      <preserveFixedJoint>true</preserveFixedJoint>
-    </gazebo>
-  </xacro:unless>
-  <!-- CAMERA -->
-  <xacro:unless value="${bringup}">
-    <link name="camera_link">
-      <collision>
-        <origin xyz="0 0 0" rpy="0 0 0"/>
-        <geometry>
-          <box size="0.05 0.05 0.05"/>
-        </geometry>
-      </collision>
-      <visual>
-        <origin xyz="0 0 0" rpy="0 0 0"/>
-        <geometry>
-          <box size="0.05 0.05 0.05"/>
-        </geometry>
-      </visual>
-      <inertial>
-        <mass value="1.0" />
-        <origin xyz="0 0 0" rpy="0 0 0"/>
-        <inertia ixx="0.0" ixy="0.0" ixz="0.0" iyy="0.0" iyz="0.0" izz="0.0" />
-      </inertial>
-    </link>
-    <joint name="camera_joint" type="fixed">
-      <origin xyz="0.776 0.526 1.90" rpy="0 1.23 3.1416"/>
-      <parent link="world"/>
-      <child link="camera_link"/>
-    </joint>
-    <gazebo reference="camera_link">
-      <sensor name="camera" type="camera">
-        <update_rate>30</update_rate>
-        <camera name="head">
-          <horizontal_fov>1.22</horizontal_fov>
-          <image>
-            <width>1920</width>
-            <height>1080</height>
-            <format>R8G8B8</format>
-          </image>
-          <clip>
-            <near>0.02</near>
-            <far>300</far>
-          </clip>
-          <noise>
-            <type>gaussian</type>
-            <mean>0.0</mean>
-            <stddev>0.007</stddev>
-          </noise>
-        </camera>
-        <plugin filename="libgazebo_ros_camera.so" name="camera_controller">
-          <robotNamespace/>
-          <alwaysOn>true</alwaysOn>
-          <updateRate>0.0</updateRate>
-          <cameraName>camera</cameraName>
-          <imageTopicName>image_raw</imageTopicName>
-          <cameraInfoTopicName>camera_info</cameraInfoTopicName>
-          <frameName>camera</frameName>
-          <hackBaseline>0.07</hackBaseline>
-        </plugin>
-      </sensor>
-    </gazebo>
-  </xacro:unless>
 </robot>

File: irb120cranfield/urdf/irb120cranfield_3.urdf.xacro (robot description, xacro)
@@ -72,5 +72,5 @@
       <origin xyz="0.0 0.0 0.0" rpy="0 0 0" />
       <geometry>
-        <mesh filename="file://$(find irb120cranfield_gazebo)/meshes/irb120enclosure/IRB120enclosure.dae" scale="1 1 1" />
+        <mesh filename="file://$(find irb120cranfield)/meshes/irb120enclosure/IRB120enclosure.dae" scale="1 1 1" />
       </geometry>
     </visual>
@@ -78,5 +78,5 @@
       <origin xyz="0.0 0.0 0.0" rpy="0 0 0" />
       <geometry>
-        <mesh filename="file://$(find irb120cranfield_gazebo)/meshes/irb120enclosure/IRB120enclosure.dae" scale="1 1 1" />
+        <mesh filename="file://$(find irb120cranfield)/meshes/irb120enclosure/IRB120enclosure.dae" scale="1 1 1" />
       </geometry>
     </collision>
@@ -103,5 +103,5 @@
       <origin xyz="0.0 0.0 0.0" rpy="0 0 0" />
       <geometry>
-        <mesh filename="file://$(find irb120cranfield_gazebo)/meshes/irb120enclosure/ergobox.dae" scale="1 1 1" />
+        <mesh filename="file://$(find irb120cranfield)/meshes/irb120enclosure/ergobox.dae" scale="1 1 1" />
       </geometry>
     </visual>
@@ -109,5 +109,5 @@
       <origin xyz="0.0 0.0 0.0" rpy="0 0 0" />
       <geometry>
-        <mesh filename="file://$(find irb120cranfield_gazebo)/meshes/irb120enclosure/ergobox.dae" scale="1 1 1" />
+        <mesh filename="file://$(find irb120cranfield)/meshes/irb120enclosure/ergobox.dae" scale="1 1 1" />
       </geometry>
     </collision>
@@ -123,3 +123,92 @@
     <origin xyz="0.0 0.0 0.0" rpy="0.0 0.0 0.0" />
   </joint>
+  <!-- ARUCO TAG -->
+  <xacro:unless value="${bringup}">
+    <!-- ARUCO GRID -->
+    <link name="aruco_grid">
+      <visual>
+        <origin xyz="0.0 0.0 0.0" rpy="0 0 0" />
+        <geometry>
+          <mesh filename="file://$(find irb120cranfield)/meshes/aruco/arucoGrid.dae" scale="1 1 1" />
+        </geometry>
+      </visual>
+      <collision>
+        <origin xyz="0.0 0.0 0.0" rpy="0 0 0" />
+        <geometry>
+          <mesh filename="file://$(find irb120cranfield)/meshes/aruco/arucoGrid.dae" scale="1 1 1" />
+        </geometry>
+      </collision>
+      <inertial>
+        <mass value="10.0"/>
+        <inertia ixx="0.0002" ixy="0.0002" ixz="0.0002" iyy="0.0" iyz="0.0" izz="0.0" />
+      </inertial>
+    </link>
+    <joint name="cell-aruco_grid-fixed" type="fixed">
+      <parent link="cell"/>
+      <child link="aruco_grid"/>
+      <origin xyz="0.0 0.0 0.0" rpy="0.0 0.0 0.0" />
+    </joint>
+    <gazebo reference="cell-aruco_grid-fixed">
+      <preserveFixedJoint>true</preserveFixedJoint>
+    </gazebo>
+  </xacro:unless>
+  <!-- CAMERA -->
+  <xacro:unless value="${bringup}">
+    <link name="camera_link">
+      <collision>
+        <origin xyz="0 0 0" rpy="0 0 0"/>
+        <geometry>
+          <box size="0.05 0.05 0.05"/>
+        </geometry>
+      </collision>
+      <visual>
+        <origin xyz="0 0 0" rpy="0 0 0"/>
+        <geometry>
+          <box size="0.05 0.05 0.05"/>
+        </geometry>
+      </visual>
+      <inertial>
+        <mass value="1.0" />
+        <origin xyz="0 0 0" rpy="0 0 0"/>
+        <inertia ixx="0.0" ixy="0.0" ixz="0.0" iyy="0.0" iyz="0.0" izz="0.0" />
+      </inertial>
+    </link>
+    <joint name="camera_joint" type="fixed">
+      <origin xyz="0.776 0.526 1.90" rpy="0 1.23 3.1416"/>
+      <parent link="world"/>
+      <child link="camera_link"/>
+    </joint>
+    <gazebo reference="camera_link">
+      <sensor name="camera" type="camera">
+        <update_rate>30</update_rate>
+        <camera name="head">
+          <horizontal_fov>1.22</horizontal_fov>
+          <image>
+            <width>1920</width>
+            <height>1080</height>
+            <format>R8G8B8</format>
+          </image>
+          <clip>
+            <near>0.02</near>
+            <far>300</far>
+          </clip>
+          <noise>
+            <type>gaussian</type>
+            <mean>0.0</mean>
+            <stddev>0.007</stddev>
+          </noise>
+        </camera>
+        <plugin filename="libgazebo_ros_camera.so" name="camera_controller">
+          <robotNamespace/>
+          <alwaysOn>true</alwaysOn>
+          <updateRate>0.0</updateRate>
+          <cameraName>camera</cameraName>
+          <imageTopicName>image_raw</imageTopicName>
+          <cameraInfoTopicName>camera_info</cameraInfoTopicName>
+          <frameName>camera</frameName>
+          <hackBaseline>0.07</hackBaseline>
+        </plugin>
+      </sensor>
+    </gazebo>
+  </xacro:unless>
 </robot>

File: irb120cranfield/urdf/objects/BlackCube.urdf (robot description, URDF)
Before this commit: robot cube, 1 links, 0 joints
Links:
- link ${name}: geometry collision mesh filename=file://$(find irb120cranfield)/meshes/objects/${name}.dae; visual mesh filename=file://$(find irb120cranfield)/meshes/objects/${name}.dae

Commit message: Migrate IRB120-CranfieldUni to GzFortress.

File: irb120cranfield/urdf/irb120cranfield_1.urdf.xacro (robot description, xacro)
@@ -50,6 +50,5 @@
   <xacro:unless value="${bringup}">
     <gazebo>
-      <plugin filename="libgazebo_ros2_control.so" name="gazebo_ros2_control">
-        <robot_sim_type>gazebo_ros2_control/GazeboSystem</robot_sim_type>
+      <plugin filename="gz_ros2_control-system" name="gz_ros2_control::GazeboSimROS2ControlPlugin">
         <!-- IRB120 Controller -->
         <parameters>$(find ros2srrc_robots)/irb120/config/controller.yaml</parameters>
@@ -70,10 +69,10 @@
       <origin xyz="0.0 0.0 0.0" rpy="0 0 0" />
       <geometry>
-        <mesh filename="file://$(find irb120cranfield)/meshes/irb120enclosure/IRB120enclosure.dae" scale="1 1 1" />
+        <mesh filename="file://$(find irb120cranfield)/meshes/irb120enclosure/IRB120enclosure.stl" scale="1 1 1" />
       </geometry>
     </collision>
     <inertial>
       <mass value="1000.0"/>
-      <inertia ixx="500.0" ixy="500.0" ixz="500.0" iyy="500.0" iyz="500.0" izz="500.0" />
+      <inertia ixx="200.0" ixy="0.0" ixz="0.0" iyy="200.0" iyz="0.0" izz="200.0"/>
     </inertial>
   </link>

File: irb120cranfield/urdf/irb120cranfield_2.urdf.xacro (robot description, xacro)
@@ -56,6 +56,5 @@
   <xacro:unless value="${bringup}">
     <gazebo>
-      <plugin filename="libgazebo_ros2_control.so" name="gazebo_ros2_control">
-        <robot_sim_type>gazebo_ros2_control/GazeboSystem</robot_sim_type>
+      <plugin filename="gz_ros2_control-system" name="gz_ros2_control::GazeboSimROS2ControlPlugin">
         <!-- IRB120 Controller -->
         <parameters>$(find ros2srrc_robots)/irb120/config/controller.yaml</parameters>
@@ -78,10 +77,10 @@
       <origin xyz="0.0 0.0 0.0" rpy="0 0 0" />
       <geometry>
-        <mesh filename="file://$(find irb120cranfield)/meshes/irb120enclosure/IRB120enclosure.dae" scale="1 1 1" />
+        <mesh filename="file://$(find irb120cranfield)/meshes/irb120enclosure/IRB120enclosure.stl" scale="1 1 1" />
       </geometry>
     </collision>
     <inertial>
       <mass value="1000.0"/>
-      <inertia ixx="500.0" ixy="500.0" ixz="500.0" iyy="500.0" iyz="500.0" izz="500.0" />
+      <inertia ixx="200.0" ixy="0.0" ixz="0.0" iyy="200.0" iyz="0.0" izz="200.0"/>
     </inertial>
   </link>
@@ -114,5 +113,5 @@
     <inertial>
       <mass value="10.0"/>
-      <inertia ixx="500.0" ixy="500.0" ixz="500.0" iyy="500.0" iyz="500.0" izz="500.0" />
+      <inertia ixx="200.0" ixy="0.0" ixz="0.0" iyy="200.0" iyz="0.0" izz="200.0"/>
     </inertial>
   </link>

File: irb120cranfield/urdf/irb120cranfield_3.urdf.xacro (robot description, xacro)
@@ -56,6 +56,5 @@
   <xacro:unless value="${bringup}">
     <gazebo>
-      <plugin filename="libgazebo_ros2_control.so" name="gazebo_ros2_control">
-        <robot_sim_type>gazebo_ros2_control/GazeboSystem</robot_sim_type>
+      <plugin filename="gz_ros2_control-system" name="gz_ros2_control::GazeboSimROS2ControlPlugin">
         <!-- IRB120 Controller -->
         <parameters>$(find ros2srrc_robots)/irb120/config/controller.yaml</parameters>
@@ -78,10 +77,10 @@
       <origin xyz="0.0 0.0 0.0" rpy="0 0 0" />
       <geometry>
-        <mesh filename="file://$(find irb120cranfield)/meshes/irb120enclosure/IRB120enclosure.dae" scale="1 1 1" />
+        <mesh filename="file://$(find irb120cranfield)/meshes/irb120enclosure/IRB120enclosure.stl" scale="1 1 1" />
       </geometry>
     </collision>
     <inertial>
       <mass value="1000.0"/>
-      <inertia ixx="500.0" ixy="500.0" ixz="500.0" iyy="500.0" iyz="500.0" izz="500.0" />
+      <inertia ixx="200.0" ixy="0.0" ixz="0.0" iyy="200.0" iyz="0.0" izz="200.0"/>
     </inertial>
   </link>
@@ -114,5 +113,5 @@
     <inertial>
       <mass value="10.0"/>
-      <inertia ixx="500.0" ixy="500.0" ixz="500.0" iyy="500.0" iyz="500.0" izz="500.0" />
+      <inertia ixx="200.0" ixy="0.0" ixz="0.0" iyy="200.0" iyz="0.0" izz="200.0"/>
     </inertial>
   </link>
@@ -133,13 +132,7 @@
         </geometry>
       </visual>
-      <collision>
-        <origin xyz="0.0 0.0 0.0" rpy="0 0 0" />
-        <geometry>
-          <mesh filename="file://$(find irb120cranfield)/meshes/aruco/arucoGrid.dae" scale="1 1 1" />
-        </geometry>
-      </collision>
       <inertial>
         <mass value="10.0"/>
-        <inertia ixx="0.0002" ixy="0.0002" ixz="0.0002" iyy="0.0" iyz="0.0" izz="0.0" />
+        <inertia ixx="0.04" ixy="0.0" ixz="0.0" iyy="0.04" iyz="0.0" izz="0.04"/>
       </inertial>
     </link>
@@ -171,5 +164,5 @@
         <mass value="1.0" />
         <origin xyz="0 0 0" rpy="0 0 0"/>
-        <inertia ixx="0.0" ixy="0.0" ixz="0.0" iyy="0.0" iyz="0.0" izz="0.0" />
+        <inertia ixx="0.0005" ixy="0.0" ixz="0.0" iyy="0.0005" iyz="0.0" izz="0.0005"/>
       </inertial>
     </link>
@@ -181,5 +174,10 @@
     <gazebo reference="camera_link">
       <sensor name="camera" type="camera">
+        <pose>0 0 0 0 0 0</pose>
+        <always_on>true</always_on>
         <update_rate>30</update_rate>
+        <visualize>true</visualize>
+        <!-- Gz Transport topic -->
+        <topic>/camera/image_raw</topic>
         <camera name="head">
           <horizontal_fov>1.22</horizontal_fov>
@@ -189,24 +187,7 @@
             <format>R8G8B8</format>
           </image>
-          <clip>
-            <near>0.02</near>
-            <far>300</far>
-          </clip>
-          <noise>
-            <type>gaussian</type>
-            <mean>0.0</mean>
-            <stddev>0.007</stddev>
-          </noise>
+          <clip><near>0.02</near><far>300</far></clip>
+          <camera_info_topic>/camera/camera_info</camera_info_topic>
         </camera>
-        <plugin filename="libgazebo_ros_camera.so" name="camera_controller">
-          <robotNamespace/>
-          <alwaysOn>true</alwaysOn>
-          <updateRate>0.0</updateRate>
-          <cameraName>camera</cameraName>
-          <imageTopicName>image_raw</imageTopicName>
-          <cameraInfoTopicName>camera_info</cameraInfoTopicName>
-          <frameName>camera</frameName>
-          <hackBaseline>0.07</hackBaseline>
-        </plugin>
       </sensor>
     </gazebo>

File: irb120cranfield/urdf/objects/BlackCube.urdf (robot description, URDF)
Before this commit: robot cube, 1 links, 0 joints
Links:
- link ${name}: geometry collision mesh filename=file://$(find irb120cranfield)/meshes/objects/BlackCube.dae; visual mesh filename=file://$(find irb120cranfield)/meshes/objects/BlackCube.dae

File: irb120cranfield/urdf/objects/BlueCube.urdf (robot description, URDF)
Before this commit: robot cube, 1 links, 0 joints
Links:
- link ${name}: geometry collision mesh filename=file://$(find irb120cranfield)/meshes/objects/BlueCube.dae; visual mesh filename=file://$(find irb120cranfield)/meshes/objects/BlueCube.dae

File: irb120cranfield/urdf/objects/GreenCube.urdf (robot description, URDF)
Before this commit: robot cube, 1 links, 0 joints
Links:
- link ${name}: geometry collision mesh filename=file://$(find irb120cranfield)/meshes/objects/GreenCube.dae; visual mesh filename=file://$(find irb120cranfield)/meshes/objects/GreenCube.dae

File: irb120cranfield/urdf/objects/RedCube.urdf (robot description, URDF)
Before this commit: robot cube, 1 links, 0 joints
Links:
- link ${name}: geometry collision mesh filename=file://$(find irb120cranfield)/meshes/objects/RedCube.dae; visual mesh filename=file://$(find irb120cranfield)/meshes/objects/RedCube.dae

File: irb120cranfield/urdf/objects/WhiteCube.urdf (robot description, URDF)
Before this commit: robot cube, 1 links, 0 joints
Links:
- link ${name}: geometry collision mesh filename=file://$(find irb120cranfield)/meshes/objects/WhiteCube.dae; visual mesh filename=file://$(find irb120cranfield)/meshes/objects/WhiteCube.dae
