Commit message: Add {prefix} to robot urdf files.

File: irb120cranfield/urdf/irb120cranfield_1.urdf.xacro (robot description, xacro)
@@ -39,4 +39,6 @@
   <xacro:arg name="EE_name" default="none"/>
   <xacro:property name="EE_name" value="$(arg EE_name)"/>
+  <xacro:arg name="prefix" default=""/>
+  <xacro:property name="prefix" value="$(arg prefix)"/>
   <!-- Include XACRO-MACRO file of the IRB120: -->
   <xacro:include filename="$(find ros2srrc_robots)/irb120/urdf/irb120_macro.urdf.xacro"/>
@@ -46,4 +48,5 @@
     EE="${EE}"
     EE_name="${EE_name}"
+    prefix="${prefix}"
   />
   <!-- Load ROS 2 Gazebo Plugin -->
@@ -60,5 +63,5 @@
   <link name="world"/>
   <!-- ABB IRB-120 ENCLOSURE -->
-  <link name="cell">
+  <link name="${prefix}cell">
     <visual>
       <origin xyz="0.0 0.0 0.0" rpy="0 0 0" />
@@ -79,13 +82,13 @@
   </link>
   <!-- Robot Cell: FIXED JOINT -->
-  <joint name="world-cell-fixed" type="fixed">
+  <joint name="${prefix}world-cell-fixed" type="fixed">
     <parent link="world"/>
-    <child link="cell"/>
+    <child link="${prefix}cell"/>
     <origin xyz="0.926 -0.124 0.0" rpy="0.0 0.0 0.0" />
   </joint>
   <!-- Robot+Cell JOINT -->
-  <joint name="cell-base_link-fixed" type="fixed">
-    <parent link="cell"/>
-    <child link="base_link"/>
+  <joint name="${prefix}cell-base_link-fixed" type="fixed">
+    <parent link="${prefix}cell"/>
+    <child link="${prefix}base_link"/>
     <origin xyz="-0.6506 0.6489 0.8605" rpy="0.0 0.0 0.0" />
   </joint>

File: irb120cranfield/urdf/irb120cranfield_2.urdf.xacro (robot description, xacro)
@@ -39,4 +39,6 @@
   <xacro:arg name="EE_name" default="none"/>
   <xacro:property name="EE_name" value="$(arg EE_name)"/>
+  <xacro:arg name="prefix" default=""/>
+  <xacro:property name="prefix" value="$(arg prefix)"/>
   <!-- Include XACRO-MACRO file of the IRB120: -->
   <xacro:include filename="$(find ros2srrc_robots)/irb120/urdf/irb120_macro.urdf.xacro"/>
@@ -46,4 +48,5 @@
     EE="${EE}"
     EE_name="${EE_name}"
+    prefix="${prefix}"
   />
   <!-- Include XACRO-MACRO file of the EGP64: -->
@@ -51,5 +54,6 @@
   <xacro:egp64
     bringup="${bringup}"
-    parent_link="tool0"
+    parent_link="${prefix}tool0"
+    prefix="${prefix}"
   />
   <!-- Load ROS 2 Gazebo Plugin -->
@@ -68,5 +72,5 @@
   <link name="world"/>
   <!-- ABB IRB-120 ENCLOSURE -->
-  <link name="cell">
+  <link name="${prefix}cell">
     <visual>
       <origin xyz="0.0 0.0 0.0" rpy="0 0 0" />
@@ -87,17 +91,17 @@
   </link>
   <!-- Robot Cell: FIXED JOINT -->
-  <joint name="world-cell-fixed" type="fixed">
+  <joint name="${prefix}world-cell-fixed" type="fixed">
     <parent link="world"/>
-    <child link="cell"/>
+    <child link="${prefix}cell"/>
     <origin xyz="0.926 -0.124 0.0" rpy="0.0 0.0 0.0" />
   </joint>
   <!-- Robot+Cell JOINT -->
-  <joint name="cell-base_link-fixed" type="fixed">
-    <parent link="cell"/>
-    <child link="base_link"/>
+  <joint name="${prefix}cell-base_link-fixed" type="fixed">
+    <parent link="${prefix}cell"/>
+    <child link="${prefix}base_link"/>
     <origin xyz="-0.6506 0.6489 0.8605" rpy="0.0 0.0 0.0" />
   </joint>
   <!-- ERGOBOX -->
-  <link name="ergobox">
+  <link name="${prefix}ergobox">
     <visual>
       <origin xyz="0.0 0.0 0.0" rpy="0 0 0" />
@@ -118,7 +122,7 @@
   </link>
   <!-- Ergobox: FIXED JOINT -->
-  <joint name="ergobox-cell-fixed" type="fixed">
-    <parent link="cell"/>
-    <child link="ergobox"/>
+  <joint name="${prefix}ergobox-cell-fixed" type="fixed">
+    <parent link="${prefix}cell"/>
+    <child link="${prefix}ergobox"/>
     <origin xyz="0.0 0.0 0.0" rpy="0.0 0.0 0.0" />
   </joint>

File: irb120cranfield/urdf/irb120cranfield_3.urdf.xacro (robot description, xacro)
@@ -39,4 +39,6 @@
   <xacro:arg name="EE_name" default="none"/>
   <xacro:property name="EE_name" value="$(arg EE_name)"/>
+  <xacro:arg name="prefix" default=""/>
+  <xacro:property name="prefix" value="$(arg prefix)"/>
   <!-- Include XACRO-MACRO file of the IRB120: -->
   <xacro:include filename="$(find ros2srrc_robots)/irb120/urdf/irb120_macro.urdf.xacro"/>
@@ -46,4 +48,5 @@
     EE="${EE}"
     EE_name="${EE_name}"
+    prefix="${prefix}"
   />
   <!-- Include XACRO-MACRO file of the EGP64: -->
@@ -51,5 +54,6 @@
   <xacro:egp64
     bringup="${bringup}"
-    parent_link="tool0"
+    parent_link="${prefix}tool0"
+    prefix="${prefix}"
   />
   <!-- Load ROS 2 Gazebo Plugin -->
@@ -68,5 +72,5 @@
   <link name="world"/>
   <!-- ABB IRB-120 ENCLOSURE -->
-  <link name="cell">
+  <link name="${prefix}cell">
     <visual>
       <origin xyz="0.0 0.0 0.0" rpy="0 0 0" />
@@ -87,17 +91,17 @@
   </link>
   <!-- Robot Cell: FIXED JOINT -->
-  <joint name="world-cell-fixed" type="fixed">
+  <joint name="${prefix}world-cell-fixed" type="fixed">
     <parent link="world"/>
-    <child link="cell"/>
+    <child link="${prefix}cell"/>
     <origin xyz="0.926 -0.124 0.0" rpy="0.0 0.0 0.0" />
   </joint>
   <!-- Robot+Cell JOINT -->
-  <joint name="cell-base_link-fixed" type="fixed">
-    <parent link="cell"/>
-    <child link="base_link"/>
+  <joint name="${prefix}cell-base_link-fixed" type="fixed">
+    <parent link="${prefix}cell"/>
+    <child link="${prefix}base_link"/>
     <origin xyz="-0.6506 0.6489 0.8605" rpy="0.0 0.0 0.0" />
   </joint>
   <!-- ERGOBOX -->
-  <link name="ergobox">
+  <link name="${prefix}ergobox">
     <visual>
       <origin xyz="0.0 0.0 0.0" rpy="0 0 0" />
@@ -118,7 +122,7 @@
   </link>
   <!-- Ergobox: FIXED JOINT -->
-  <joint name="ergobox-cell-fixed" type="fixed">
-    <parent link="cell"/>
-    <child link="ergobox"/>
+  <joint name="${prefix}ergobox-cell-fixed" type="fixed">
+    <parent link="${prefix}cell"/>
+    <child link="${prefix}ergobox"/>
     <origin xyz="0.0 0.0 0.0" rpy="0.0 0.0 0.0" />
   </joint>
@@ -126,5 +130,5 @@
   <xacro:unless value="${bringup}">
     <!-- ARUCO GRID -->
-    <link name="aruco_grid">
+    <link name="${prefix}aruco_grid">
       <visual>
         <origin xyz="0.0 0.0 0.0" rpy="0 0 0" />
@@ -144,10 +148,10 @@
       </inertial>
     </link>
-    <joint name="cell-aruco_grid-fixed" type="fixed">
-      <parent link="cell"/>
-      <child link="aruco_grid"/>
+    <joint name="${prefix}cell-aruco_grid-fixed" type="fixed">
+      <parent link="${prefix}cell"/>
+      <child link="${prefix}aruco_grid"/>
       <origin xyz="0.0 0.0 0.0" rpy="0.0 0.0 0.0" />
     </joint>
-    <gazebo reference="cell-aruco_grid-fixed">
+    <gazebo reference="${prefix}cell-aruco_grid-fixed">
       <preserveFixedJoint>true</preserveFixedJoint>
     </gazebo>
@@ -155,5 +159,5 @@
   <!-- CAMERA -->
   <xacro:unless value="${bringup}">
-    <link name="camera_link">
+    <link name="${prefix}camera_link">
       <collision>
         <origin xyz="0 0 0" rpy="0 0 0"/>
@@ -174,10 +178,10 @@
       </inertial>
     </link>
-    <joint name="camera_joint" type="fixed">
+    <joint name="${prefix}camera_joint" type="fixed">
       <origin xyz="0.776 0.526 1.90" rpy="0 1.23 3.1416"/>
       <parent link="world"/>
-      <child link="camera_link"/>
+      <child link="${prefix}camera_link"/>
     </joint>
-    <gazebo reference="camera_link">
+    <gazebo reference="${prefix}camera_link">
       <sensor name="camera" type="camera">
         <update_rate>30</update_rate>

Commit message: Add (prefix) to urdf files.

File: irb120cranfield/urdf/irb120cranfield_1.urdf.xacro (robot description, xacro)
@@ -39,4 +39,6 @@
   <xacro:arg name="EE_name" default="none"/>
   <xacro:property name="EE_name" value="$(arg EE_name)"/>
+  <xacro:arg name="prefix" default=""/>
+  <xacro:property name="prefix" value="$(arg prefix)"/>
   <!-- Include XACRO-MACRO file of the IRB120: -->
   <xacro:include filename="$(find ros2srrc_robots)/irb120/urdf/irb120_macro.urdf.xacro"/>
@@ -46,4 +48,5 @@
     EE="${EE}"
     EE_name="${EE_name}"
+    prefix="${prefix}"
   />
   <!-- Load ROS 2 Gazebo Plugin -->
@@ -59,5 +62,5 @@
   <link name="world"/>
   <!-- ABB IRB-120 ENCLOSURE -->
-  <link name="cell">
+  <link name="${prefix}cell">
     <visual>
       <origin xyz="0.0 0.0 0.0" rpy="0 0 0" />
@@ -78,13 +81,13 @@
   </link>
   <!-- Robot Cell: FIXED JOINT -->
-  <joint name="world-cell-fixed" type="fixed">
+  <joint name="${prefix}world-cell-fixed" type="fixed">
     <parent link="world"/>
-    <child link="cell"/>
+    <child link="${prefix}cell"/>
     <origin xyz="0.926 -0.124 0.0" rpy="0.0 0.0 0.0" />
   </joint>
   <!-- Robot+Cell JOINT -->
-  <joint name="cell-base_link-fixed" type="fixed">
-    <parent link="cell"/>
-    <child link="base_link"/>
+  <joint name="${prefix}cell-base_link-fixed" type="fixed">
+    <parent link="${prefix}cell"/>
+    <child link="${prefix}base_link"/>
     <origin xyz="-0.6506 0.6489 0.8605" rpy="0.0 0.0 0.0" />
   </joint>

File: irb120cranfield/urdf/irb120cranfield_2.urdf.xacro (robot description, xacro)
@@ -39,4 +39,6 @@
   <xacro:arg name="EE_name" default="none"/>
   <xacro:property name="EE_name" value="$(arg EE_name)"/>
+  <xacro:arg name="prefix" default=""/>
+  <xacro:property name="prefix" value="$(arg prefix)"/>
   <!-- Include XACRO-MACRO file of the IRB120: -->
   <xacro:include filename="$(find ros2srrc_robots)/irb120/urdf/irb120_macro.urdf.xacro"/>
@@ -46,4 +48,5 @@
     EE="${EE}"
     EE_name="${EE_name}"
+    prefix="${prefix}"
   />
   <!-- Include XACRO-MACRO file of the EGP64: -->
@@ -51,5 +54,6 @@
   <xacro:egp64
     bringup="${bringup}"
-    parent_link="tool0"
+    parent_link="${prefix}tool0"
+    prefix="${prefix}"
   />
   <!-- Load ROS 2 Gazebo Plugin -->
@@ -67,5 +71,5 @@
   <link name="world"/>
   <!-- ABB IRB-120 ENCLOSURE -->
-  <link name="cell">
+  <link name="${prefix}cell">
     <visual>
       <origin xyz="0.0 0.0 0.0" rpy="0 0 0" />
@@ -86,17 +90,17 @@
   </link>
   <!-- Robot Cell: FIXED JOINT -->
-  <joint name="world-cell-fixed" type="fixed">
+  <joint name="${prefix}world-cell-fixed" type="fixed">
     <parent link="world"/>
-    <child link="cell"/>
+    <child link="${prefix}cell"/>
     <origin xyz="0.926 -0.124 0.0" rpy="0.0 0.0 0.0" />
   </joint>
   <!-- Robot+Cell JOINT -->
-  <joint name="cell-base_link-fixed" type="fixed">
-    <parent link="cell"/>
-    <child link="base_link"/>
+  <joint name="${prefix}cell-base_link-fixed" type="fixed">
+    <parent link="${prefix}cell"/>
+    <child link="${prefix}base_link"/>
     <origin xyz="-0.6506 0.6489 0.8605" rpy="0.0 0.0 0.0" />
   </joint>
   <!-- ERGOBOX -->
-  <link name="ergobox">
+  <link name="${prefix}ergobox">
     <visual>
       <origin xyz="0.0 0.0 0.0" rpy="0 0 0" />
@@ -117,7 +121,7 @@
   </link>
   <!-- Ergobox: FIXED JOINT -->
-  <joint name="ergobox-cell-fixed" type="fixed">
-    <parent link="cell"/>
-    <child link="ergobox"/>
+  <joint name="${prefix}ergobox-cell-fixed" type="fixed">
+    <parent link="${prefix}cell"/>
+    <child link="${prefix}ergobox"/>
     <origin xyz="0.0 0.0 0.0" rpy="0.0 0.0 0.0" />
   </joint>

File: irb120cranfield/urdf/irb120cranfield_3.urdf.xacro (robot description, xacro)
@@ -39,4 +39,6 @@
   <xacro:arg name="EE_name" default="none"/>
   <xacro:property name="EE_name" value="$(arg EE_name)"/>
+  <xacro:arg name="prefix" default=""/>
+  <xacro:property name="prefix" value="$(arg prefix)"/>
   <!-- Include XACRO-MACRO file of the IRB120: -->
   <xacro:include filename="$(find ros2srrc_robots)/irb120/urdf/irb120_macro.urdf.xacro"/>
@@ -46,4 +48,5 @@
     EE="${EE}"
     EE_name="${EE_name}"
+    prefix="${prefix}"
   />
   <!-- Include XACRO-MACRO file of the EGP64: -->
@@ -51,5 +54,6 @@
   <xacro:egp64
     bringup="${bringup}"
-    parent_link="tool0"
+    parent_link="${prefix}tool0"
+    prefix="${prefix}"
   />
   <!-- Load ROS 2 Gazebo Plugin -->
@@ -67,5 +71,5 @@
   <link name="world"/>
   <!-- ABB IRB-120 ENCLOSURE -->
-  <link name="cell">
+  <link name="${prefix}cell">
     <visual>
       <origin xyz="0.0 0.0 0.0" rpy="0 0 0" />
@@ -86,17 +90,17 @@
   </link>
   <!-- Robot Cell: FIXED JOINT -->
-  <joint name="world-cell-fixed" type="fixed">
+  <joint name="${prefix}world-cell-fixed" type="fixed">
     <parent link="world"/>
-    <child link="cell"/>
+    <child link="${prefix}cell"/>
     <origin xyz="0.926 -0.124 0.0" rpy="0.0 0.0 0.0" />
   </joint>
   <!-- Robot+Cell JOINT -->
-  <joint name="cell-base_link-fixed" type="fixed">
-    <parent link="cell"/>
-    <child link="base_link"/>
+  <joint name="${prefix}cell-base_link-fixed" type="fixed">
+    <parent link="${prefix}cell"/>
+    <child link="${prefix}base_link"/>
     <origin xyz="-0.6506 0.6489 0.8605" rpy="0.0 0.0 0.0" />
   </joint>
   <!-- ERGOBOX -->
-  <link name="ergobox">
+  <link name="${prefix}ergobox">
     <visual>
       <origin xyz="0.0 0.0 0.0" rpy="0 0 0" />
@@ -117,7 +121,7 @@
   </link>
   <!-- Ergobox: FIXED JOINT -->
-  <joint name="ergobox-cell-fixed" type="fixed">
-    <parent link="cell"/>
-    <child link="ergobox"/>
+  <joint name="${prefix}ergobox-cell-fixed" type="fixed">
+    <parent link="${prefix}cell"/>
+    <child link="${prefix}ergobox"/>
     <origin xyz="0.0 0.0 0.0" rpy="0.0 0.0 0.0" />
   </joint>
@@ -125,5 +129,5 @@
   <xacro:unless value="${bringup}">
     <!-- ARUCO GRID -->
-    <link name="aruco_grid">
+    <link name="${prefix}aruco_grid">
       <visual>
         <origin xyz="0.0 0.0 0.0" rpy="0 0 0" />
@@ -137,10 +141,10 @@
       </inertial>
     </link>
-    <joint name="cell-aruco_grid-fixed" type="fixed">
-      <parent link="cell"/>
-      <child link="aruco_grid"/>
+    <joint name="${prefix}cell-aruco_grid-fixed" type="fixed">
+      <parent link="${prefix}cell"/>
+      <child link="${prefix}aruco_grid"/>
       <origin xyz="0.0 0.0 0.0" rpy="0.0 0.0 0.0" />
     </joint>
-    <gazebo reference="cell-aruco_grid-fixed">
+    <gazebo reference="${prefix}cell-aruco_grid-fixed">
       <preserveFixedJoint>true</preserveFixedJoint>
     </gazebo>
@@ -148,5 +152,5 @@
   <!-- CAMERA -->
   <xacro:unless value="${bringup}">
-    <link name="camera_link">
+    <link name="${prefix}camera_link">
       <collision>
         <origin xyz="0 0 0" rpy="0 0 0"/>
@@ -167,11 +171,11 @@
       </inertial>
     </link>
-    <joint name="camera_joint" type="fixed">
+    <joint name="${prefix}camera_joint" type="fixed">
       <origin xyz="0.776 0.526 1.90" rpy="0 1.23 3.1416"/>
       <parent link="world"/>
-      <child link="camera_link"/>
+      <child link="${prefix}camera_link"/>
     </joint>
-    <gazebo reference="camera_link">
-      <sensor name="camera" type="camera">
+    <gazebo reference="${prefix}camera_link">
+      <sensor name="${prefix}camera" type="camera">
         <pose>0 0 0 0 0 0</pose>
         <always_on>true</always_on>
